Commit message: changed init home, modified basic objects

File: pick_and_place/urdf/objects/red_box.urdf (robot description, URDF)
Before this commit: robot red_box, 1 links, 0 joints
Links:
- link base_link: mass 0.010 -> 0.0010

File: pick_and_place/urdf/objects/red_cylinder.urdf (robot description, URDF)
Before this commit: robot red_cylinder, 1 links, 0 joints
Links:
- link base_link: mass 0.00001 -> 0.001
